Commit message: robot nav wip

File: src/robot_description/description/robot_description.urdf (robot description, URDF)
Before this commit: robot delivery_bot, 3 links, 2 joints
Links:
- link base_link: geometry visual mesh filename=package://robot_description/meshes/body_v2.STL scale=0.001 0.001 0.001

Commit message: fixed dependencies and launch files

File: src/robot_description/description/robot_description.urdf (robot description, URDF)
Before this commit: robot delivery_bot, 3 links, 2 joints
Links:
- link base_link: geometry visual mesh filename=package://robot_description/meshes/body.stl scale=0.001 0.001 0.001
Joints:
- joint camera_joint: origin xyz=0.215 0 0.05 rpy=0 0 0 -> xyz=0 0 .1 rpy=0 0 0
